Commit message: 로봇 크기 적용시킨거 rviz에도 적용

File: src/package_all/aimlab/lio-sam/launch/include/config/robot.urdf.xacro (robot description, xacro)
@@ -2,5 +2,19 @@
 <robot name="lio" xmlns:xacro="http://tixiaoshan.github.io/">
   <xacro:property name="PI" value="3.1415926535897931" />
-  <link name="chassis_link"></link>
+  <xacro:property name="robot_length_m" value="0.55" />
+  <xacro:property name="robot_width_m" value="0.60" />
+  <xacro:property name="robot_height_m" value="0.18" />
+  <material name="robot_body_blue">
+    <color rgba="0.10 0.45 0.85 0.65" />
+  </material>
+  <link name="chassis_link">
+    <visual>
+      <origin xyz="0 0 ${robot_height_m / 2.0}" rpy="0 0 0" />
+      <geometry>
+        <box size="${robot_length_m} ${robot_width_m} ${robot_height_m}" />
+      </geometry>
+      <material name="robot_body_blue" />
+    </visual>
+  </link>
   <link name="base_link"></link>
   <joint name="base_link_joint" type="fixed">

Commit message: 로봇 가로 세로 길이 반대로 되어 있는거 수정

File: src/package_all/aimlab/lio-sam/launch/include/config/robot.urdf.xacro (robot description, xacro)
@@ -2,6 +2,6 @@
 <robot name="lio" xmlns:xacro="http://tixiaoshan.github.io/">
   <xacro:property name="PI" value="3.1415926535897931" />
-  <xacro:property name="robot_length_m" value="0.55" />
-  <xacro:property name="robot_width_m" value="0.60" />
+  <xacro:property name="robot_length_m" value="0.60" />
+  <xacro:property name="robot_width_m" value="0.55" />
   <xacro:property name="robot_height_m" value="0.18" />
   <material name="robot_body_blue">

Commit message: Tune scout mini footprint and planning odom

File: src/package_all/aimlab/lio-sam/launch/include/config/robot.urdf.xacro (robot description, xacro)
@@ -2,6 +2,6 @@
 <robot name="lio" xmlns:xacro="http://tixiaoshan.github.io/">
   <xacro:property name="PI" value="3.1415926535897931" />
-  <xacro:property name="robot_length_m" value="0.60" />
-  <xacro:property name="robot_width_m" value="0.55" />
+  <xacro:property name="robot_length_m" value="0.612" />
+  <xacro:property name="robot_width_m" value="0.58" />
   <xacro:property name="robot_height_m" value="0.18" />
   <material name="robot_body_blue">

Commit message: Fix Ouster TF chain and risk-only replanner hold

File: src/package_all/aimlab/lio-sam/launch/include/config/robot.urdf.xacro (robot description, xacro)
@@ -29,7 +29,27 @@
     <origin xyz="0 0 0" rpy="0 0 0" />
   </joint>
+  <!-- Keep Ouster sensor frames connected to base_link so downstream nodes can
+       transform /ouster/points even when the driver publishes os_sensor. -->
+  <link name="os_sensor"> </link>
+  <joint name="os_sensor_joint" type="fixed">
+    <parent link="chassis_link" />
+    <child link="os_sensor" />
+    <origin xyz="0 0 0" rpy="0 0 0" />
+  </joint>
+  <link name="os_lidar"> </link>
+  <joint name="os_lidar_joint" type="fixed">
+    <parent link="os_sensor" />
+    <child link="os_lidar" />
+    <origin xyz="0 0 0" rpy="0 0 0" />
+  </joint>
+  <link name="os_imu"> </link>
+  <joint name="os_imu_joint" type="fixed">
+    <parent link="os_sensor" />
+    <child link="os_imu" />
+    <origin xyz="0 0 0" rpy="0 0 0" />
+  </joint>
   <link name="velodyne"> </link>
   <joint name="velodyne_joint" type="fixed">
-    <parent link="chassis_link" />
+    <parent link="os_lidar" />
     <child link="velodyne" />
     <origin xyz="0 0 0" rpy="0 0 0" />

Commit message: Revert "Fix Ouster TF chain and risk-only replanner hold"
This reverts commit 233a43fc5c1aab11a5502e9eb870c74abd1b1389.

File: src/package_all/aimlab/lio-sam/launch/include/config/robot.urdf.xacro (robot description, xacro)
@@ -29,27 +29,7 @@
     <origin xyz="0 0 0" rpy="0 0 0" />
   </joint>
-  <!-- Keep Ouster sensor frames connected to base_link so downstream nodes can
-       transform /ouster/points even when the driver publishes os_sensor. -->
-  <link name="os_sensor"> </link>
-  <joint name="os_sensor_joint" type="fixed">
-    <parent link="chassis_link" />
-    <child link="os_sensor" />
-    <origin xyz="0 0 0" rpy="0 0 0" />
-  </joint>
-  <link name="os_lidar"> </link>
-  <joint name="os_lidar_joint" type="fixed">
-    <parent link="os_sensor" />
-    <child link="os_lidar" />
-    <origin xyz="0 0 0" rpy="0 0 0" />
-  </joint>
-  <link name="os_imu"> </link>
-  <joint name="os_imu_joint" type="fixed">
-    <parent link="os_sensor" />
-    <child link="os_imu" />
-    <origin xyz="0 0 0" rpy="0 0 0" />
-  </joint>
   <link name="velodyne"> </link>
   <joint name="velodyne_joint" type="fixed">
-    <parent link="os_lidar" />
+    <parent link="chassis_link" />
     <child link="velodyne" />
     <origin xyz="0 0 0" rpy="0 0 0" />
